File: LEDRing.brd (EAGLE design)
At the start: 52.5 x 52.4 mm, 35 parts, among them U1 ATMEGA328P-AU, U2 MCP73831, U3 MIC5219 3.3V, U4 MMA8452Q, Y1 16MHZ

Commit message: Finished layout. Need to fix text
Parts:
- added R8: (no value), SparkFun-Passives:0603-RES
- moved C3 0.76 mm to (27.6, 37.6)
Connections:
- removed net VSS: D1.3, D10.3, D11.3, D12.3, D3.3, D4.3, D5.3, D6.3, D7.3, D8.3, D9.3
- net 5V: now also R8.2
- net GND: now also D1.3, D10.3, D11.3, D12.3, D3.3, D4.3, D5.3, D6.3, D7.3, D8.3, D9.3
- net LED_DATA: now also D1.4
- net VSTAT: now also R8.1, U1.1
Routing:
- net VSS: track 113.9 -> 0.00 mm
- net GND: track 104.8 -> 202.6 mm, vias 7 -> 11
- net LED_DATA: track 0.00 -> 59.5 mm, vias 0 -> 1
- net VSTAT: track 0.00 -> 56.1 mm, vias 0 -> 2
- net 5V: track 32.2 -> 63.7 mm, vias 0 -> 1
- net VBATT: track 200.7 -> 203.1 mm
- net N$23: track 23.6 -> 25.7 mm
- net N$15: track 32.6 -> 33.3 mm
- net N$19: track 24.3 -> 24.9 mm

Commit message: Sent board to be made
Other:
- board text added: "Diego Aguilera 17 Nov 2016"
- board text added: "LED Ring"
- board text added: "v1.0"
