File: HW/LEDRing.brd (EAGLE design)
At the start: 50.6 x 50.6 mm, 48 parts, among them U1 ATMEGA328P-AU, U2 MCP73831, U3 MIC5219 3.3V, U4 MMA8452Q, U5 FT231XS, Y1 16MHZ

Commit message: Updating all files. I've started adding a motor driver (vibration motor).
Parts:
- added C10, C9: 1uF, microbuilder:0805-NO
- added TP2, TP3: (no value), microbuilder:TESTPOINT_PAD_2MM
- added U$13: (no value), microbuilder:SYMBOL_MINUS
- added U$5: (no value), microbuilder:SYMBOL_PLUS
- added U6: DRV2605LDGS, microbuilder:PSOP10
Connections:
- new net IN/TRIG: U6.4
- new net N$32: C9.2, U6.1
- new net N$36: C10.1, U6.10, U6.6
- new net N$37: U6.5
- new net OUT+: TP2.P$1, U6.7
- new net OUT-: TP3.P$1, U6.9
- net GND: now also C10.2, C9.1, U6.8
- net SCL: now also U6.2
- net SDA: now also U6.3
Routing:
- net N$36: track 0.00 -> 13.4 mm
- net GND: track 198.8 -> 207.9 mm, vias 16 -> 17
- net IN/TRIG: track 0.00 -> 5.96 mm, vias 0 -> 1
- net OUT+: track 0.00 -> 4.97 mm, vias 0 -> 1
- net OUT-: track 0.00 -> 4.87 mm, vias 0 -> 1
- net N$32: track 0.00 -> 2.57 mm
- net SDA: track 9.36 -> 10.8 mm
Other:
- outline, holes or cut-outs redrawn
